File: xgsid-keyboard-pcb.kicad_sch (KiCad schematic)
At the start: 0 parts

Commit message: Parts 1-3
Parts:
- added C?: 1uF, symbol Device:C_Small
- added C? (x3): 0.1uF, symbol Device:C_Small
- added C? (x2): 22pF, symbol Device:C_Small
- added C?: 10uF, symbol Device:C_Small
- added R? (x2): 22, symbol Device:R_Small
- added R? (x2): 10k, symbol Device:R_Small
- added SW1: SW_Push, symbol Switch:SW_Push
- added U1: ATmega32U4-A, Package_QFP:TQFP-44_10x10mm_P0.8mm, symbol MCU_Microchip_ATmega:ATmega32U4-A
- added Y?: 16Mhz, symbol Device:Crystal_GND24_Small
Connections:
- new net: C?.1, U1.6 (UCAP)
- new net: C?.2, U1.17 (XTAL1), Y?.1
- new net: C?.2, U1.16 (XTAL2), Y?.3
- new net: R?.2, U1.4 (D+)
- new net: R?.2, SW1.2, U1.13 (~{RESET})
- new net: R?.2, U1.3 (D-)
- new net: R?.1, U1.33 (~{HWB}/PE2)
- new net +5V: C?.1, C?.1, C?.1, C?.1, R?.1, U1.14 (VCC), U1.2 (UVCC), U1.24 (AVCC), U1.34 (VCC), U1.44 (AVCC), U1.7 (VBUS)
- new net D+: R?.1
- new net D-: R?.1
- new net GND: C?.1, C?.1, C?.2, C?.2, C?.2, C?.2, C?.2, R?.2, SW1.1, U1.15 (GND), U1.23 (GND), U1.35 (GND), U1.43 (GND), U1.5 (UGND), Y?.2 (G), Y?.4 (G)
